File: Kicad Files/Cenere Mouse.kicad_pcb (KiCad board)
At the start: 4 copper layers, 47.8 x 89 mm, 114 parts, among them J1 HRO_Type-C-31-M-14, J2 BATTERY, J3 TC2030_SWD, Q1 2N7002, Q2 AO3401A, Q3 2N7002, SW1 SW_Slide_DPDT, SW2 CMI627301D07, SW3 CMI627301D07, SW4 CMI627301D07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

Commit message: Minor improvements (detailed list attached)
- Updated JST Connector to a more common PH 2.0mm one;
- Added some helpful silkscreen;
- Retouched some tracks;
- Updated schematic symbols information to help “automatically” generate JLC BOM;
- Adjusted Vias Annular ring sizes and clearances cleanup for JLC manufacturing;
- Adjusted gitgnore to include .csv and .xml to show BOM files on Github;
Parts:
- J2: value BATTERY -> PH-2A; footprint Connector_JST:JST_XH_B2B-XH-AM_1x02_P2.50mm_Vertical -> Connector_JST:JST_PH_B2B-PH-K_1x02_P2.00mm_Vertical
- SW5: value Microswitch -> Microswitch_DPI
- SW8: value SKRPACE010 -> Microswitch_Wheel
- U9: value SN74LVC1T45DW -> SN74LVC1T45DC
- moved J2 1.54 mm to (83.9, 101.7), turned to 180 degrees
Connections:
- J2 pad 1: +VBAT -> GND
- J2 pad 2: GND -> +VBAT
Routing:
- net GND: track 64.7 -> 66.6 mm, vias 578 -> 570
- net Net-(J1-VBUS-PadA4): track 36.4 -> 37.7 mm
- net +3V3: track 255.3 -> 255.6 mm, vias 26 -> 24
Other:
- board text added: "+"
- board text added: "+3V3"
- board text added: "CLK"
- board text added: "DO"
- board text added: "GND"
- board text added: "NRST"
- board text added: "SWDIO"
- board text added: "TC2030 - SOLDERING SIDE"
- board text added: "WIRED"
- board text added: "WIRELESS"
