File: Kicad Files/Microcontroller.kicad_sch (KiCad schematic)
At the start: 34 parts, among them J3 TC2030_SWD, SW8 SKRPACE010, U5 nRF52840-QIXX

Commit message: Minor improvements (detailed list attached)
- Updated JST Connector to a more common PH 2.0mm one;
- Added some helpful silkscreen;
- Retouched some tracks;
- Updated schematic symbols information to help “automatically” generate JLC BOM;
- Adjusted Vias Annular ring sizes and clearances cleanup for JLC manufacturing;
- Adjusted gitgnore to include .csv and .xml to show BOM files on Github;
Parts:
- C15, C31, C33: JLC PN C52923 -> (none); JLCPCB PN (none) -> C52923
- C26, C27, C43: JLC PN C1547 -> (none); JLCPCB PN (none) -> C1547
- C28, C29: JLC PN C1548 -> (none); JLCPCB PN (none) -> C1548
- C32: JLC PN C272875 -> (none); JLCPCB PN (none) -> C272875
- C34, C35, C39: JLC PN C23733 -> (none); JLCPCB PN (none) -> C23733
- C36, C37, C38, C42: JLCPCB PN (none) -> C307331; Manufacturer (none) -> Samsung; Part Number (none) -> CL05B104KB54PNC
- C40: JLC PN C307452 -> (none); JLCPCB PN (none) -> C307452
- C41: JLC PN C1546 -> (none); JLCPCB PN (none) -> C1546
- C46: JLC PN C307452 -> (none); JLCPCB PN (none) -> C88902; Manufacturer Samsung -> Murata; Part Number CL05C821JB5NNNC -> GJM1555C1HR80WB01D
- C47: JLC PN C307452 -> (none); JLCPCB PN (none) -> C2912277; Manufacturer Samsung -> Murata; Part Number CL05C821JB5NNNC -> GCM1555C1HR50WA16D
- C48: JLC PN C307452 -> (none); JLCPCB PN (none) -> C710805; Manufacturer Samsung -> Murata; Part Number CL05C821JB5NNNC -> GRM0335C1ER40WA01D
- C49: JLC PN C307452 -> (none); Manufacturer Samsung -> (none); Part Number CL05C821JB5NNNC -> (none)
- J3: now not fitted; now left out of the parts list
- L6: JLC PN C86752 -> (none); JLCPCB PN (none) -> C86752
- L7: JLC PN C668460 -> (none); JLCPCB PN (none) -> C668460
- L8: JLCPCB PN (none) -> C86065; Manufacturer (none) -> Murata; Part Number (none) -> LQG15HS4N7S02D
- R24: JLC PN C23164 -> (none); JLCPCB PN (none) -> C23164
- R25: JLCPCB PN (none) -> C25741; Manufacturer (none) -> UNI-ROYAL(Uniroyal Elec); Part Number (none) -> 0402WGF1003TCE
- R26: JLCPCB PN (none) -> C25867; Manufacturer (none) -> UNI-ROYAL(Uniroyal Elec); Part Number (none) -> 0402WGF1501TCE
- SW8: value SKRPACE010 -> Microswitch_Wheel; JLCPCB PN (none) -> C139797; Part Number (none) -> SKRPACE010
- U5: JLCPCB PN (none) -> C190794; Manufacturer (none) -> Nordic Semicon; Part Number (none) -> NRF52840-QIAA-R
- XL1: JLC PN C7500573 -> (none); JLCPCB PN (none) -> C7500573
- XL2: JLC PN C2965582 -> (none); JLCPCB PN (none) -> C2965582
Connections:
- no-connect marks 40 -> 47
