File: Kicad Files/Misc.kicad_sch (KiCad schematic)
At the start: 39 parts, among them Q2 AO3401A, Q3 2N7002, SW2 CMI627301D07, SW3 CMI627301D07, SW4 CMI627301D07, SW5 Microswitch, SW6 Microswitch, SW7 Microswitch, U6 PAW3395DM, U7 TTC/Kailh Encoder E103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

Commit message: Minor improvements (detailed list attached)
- Updated JST Connector to a more common PH 2.0mm one;
- Added some helpful silkscreen;
- Retouched some tracks;
- Updated schematic symbols information to help “automatically” generate JLC BOM;
- Adjusted Vias Annular ring sizes and clearances cleanup for JLC manufacturing;
- Adjusted gitgnore to include .csv and .xml to show BOM files on Github;
Parts:
- C10, C11, C12, C13, C14, C21, C23, C25, C44, C45: JLCPCB PN (none) -> C307331; Manufacturer (none) -> Samsung; Part Number (none) -> CL05B104KB54PNC
- C19: JLC PN C84494 -> (none); JLCPCB PN (none) -> C84494
- C20, C22, C50: JLC PN C95841 -> (none); JLCPCB PN (none) -> C95841
- C24: JLC PN C6119943 -> (none); JLCPCB PN (none) -> C6119943
- LED1, LED2, LED3, LED4, LED5: JLCPCB PN (none) -> C965555; Manufacturer (none) -> Worldsemi; Part Number (none) -> WS2812B-2020
- Q2: JLC PN C347476 -> (none); JLCPCB PN (none) -> C347476
- Q3: JLC PN C8545 -> (none); JLCPCB PN (none) -> C8545
- R15: JLCPCB PN (none) -> C23186; Manufacturer (none) -> UNI-ROYAL(Uniroyal Elec); Part Number (none) -> 0603WAF5101T5E
- R16, R18, R21: JLCPCB PN (none) -> C25804; Manufacturer (none) -> UNI-ROYAL(Uniroyal Elec); Part Number (none) -> 0603WAF1002T5E
- R17: JLCPCB PN (none) -> C22775; Manufacturer (none) -> UNI-ROYAL(Uniroyal Elec); Part Number (none) -> 0603WAF1000T5E
- R20: JLC PN C17729 -> (none); JLCPCB PN (none) -> C17729
- R22, R23: JLCPCB PN (none) -> C22935; Manufacturer (none) -> UNI-ROYAL(Uniroyal Elec); Part Number (none) -> 0603WAF1004T5E
- SW2, SW3, SW4: JLCPCB PN (none) -> C400268; Part Number (none) -> CMI627301D07; now left out of the parts list
- SW5: value Microswitch -> Microswitch_DPI; JLCPCB PN (none) -> C400257; Manufacturer (none) -> Kailh; Part Number (none) -> CMI126603D09; now left out of the parts list
- SW6, SW7: value Microswitch -> Microswitch_Extra
- U7: now left out of the parts list
- U9: value SN74LVC1T45DW -> SN74LVC1T45DC; JLCPCB PN (none) -> C9382; Manufacturer (none) -> Texas Instruments; Part Number (none) -> SN74LVC1T45DC
Connections:
- no-connect marks 0 -> 4
